File: schematics/RAM_ROM_Expansion/RAM_ROM_Expansion.kicad_sch (KiCad schematic)
At the start: 22 parts, among them P1 Cartridge Port, SW1 ROM A13, SW2 ROM A14, SW3 RAM Start, U1 62256 32K Static RAM, U2 28C256 32K EEPROM, U3 74LS00, U4 74LS02

Commit message: Add title and revision details to the schematic sheets
Other:
- title: (none) -> VZ200 / Laser-210 RAM and ROM Expansion Module
Changed lines of the file:
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@@
 (kicad_sch (version 20230121) (generator eeschema)
   (paper "A4")
+  (title_block
+    (title "VZ200 / Laser-210 RAM and ROM Expansion Module")
+    (date "2024-01-01")
+    (rev "1")
+  )
   (junction (at 124.46 154.94) (diameter 0) (color 0 0 0 0)
   )
