File: schematics/VZ200_16K_RAM_Expansion/VZ200_16K_RAM_Expansion.kicad_sch (KiCad schematic)
At the start: 18 parts, among them P2 Cartridge, U10 74LS157, U11 74LS123, U12 74LS00, U13 74LS32, U14 74LS74, U15 74LS266, U9 74LS157

Commit message: Add title and revision details to the schematic sheets
Other:
- title: (none) -> VZ200 16K Memory Expansion Module
Changed lines of the file:
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@@
 (kicad_sch (version 20230121) (generator eeschema)
   (paper "A4")
+  (title_block
+    (title "VZ200 16K Memory Expansion Module")
+    (date "2024-01-01")
+    (rev "1")
+  )
   (junction (at 106.68 143.51) (diameter 0) (color 0 0 0 0)
   )
