File: schematics/VZ200_16K_RAM_Expansion/dynamic_ram.kicad_sch (KiCad schematic)
At the start: 26 parts, among them Q1 NA31X, Q2 1502C, U1 4116, U2 4116, U3 4116, U4 4116, U5 4116, U6 4116, U7 4116, U8 4116

Commit message: Add title and revision details to the schematic sheets
Other:
- title: (none) -> VZ200 16K Memory Expansion Module
Changed lines of the file:
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@@
 (kicad_sch (version 20230121) (generator eeschema)
   (paper "A4")
+  (title_block
+    (title "VZ200 16K Memory Expansion Module")
+    (date "2024-01-01")
+    (rev "1")
+  )
   (junction (at 161.925 141.605) (diameter 0) (color 0 0 0 0)
   )
