File: schematics/VZ200_Printer_Interface/VZ200_Printer_Interface.kicad_sch (KiCad schematic)
At the start: 19 parts, among them P1 I/O Expansion, P2 Printer, U1 74LS33, U2 74LS138, U3 74LS373

Commit message: Add title and revision details to the schematic sheets
Other:
- title: (none) -> VZ200 Printer Interface
Changed lines of the file:
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@@
 (kicad_sch (version 20230121) (generator eeschema)
   (paper "A4")
+  (title_block
+    (title "VZ200 Printer Interface")
+    (date "2024-01-01")
+    (rev "1")
+  )
   (junction (at 222.25 83.82) (diameter 0) (color 0 0 0 0)
   )
